Commit message: - Modify Collada Version of Meshes - Append bringup_moveit launch file

File: safe_arm_description/urdf/safe_arm_v1.transmission.xacro (robot description, xacro)
@@ -4,6 +4,7 @@
 		<transmission name="${name}_tran">
 			<type>transmission_interface/SimpleTransmission</type>
-			<joint name="${name}">
+			<joint name="${name}" >
 				<hardwareInterface>EffortJointInterface</hardwareInterface>
+				<mechanicalReduction>1</mechanicalReduction>
 			</joint>
 			<actuator name="${name}_motor">
